File: PulseFit/PulseFit.brd (EAGLE design)
At the start: 51.5 x 57.7 mm, 47 parts, among them SW1 SWITCH.JS202011JCQN

Commit message: reorganized and regrouped repo
Parts:
- added U$2: REVISION.F, CalvEngIO-Logos:REV.F
- D1: device CalvEngIO-DiscreteSemi:SOD-323 -> CalvEngIO-DiscreteSemi:USC
- R1: value 205 -> 105
- R12: value 1.5M -> 1.47M
- R2: value 470 -> 487
- R8, R9: value 210k -> 205k
- turned D1 to 90 degrees
Connections:
- net N$10: now also D1.+; no longer D1.A
- net PEAK: now also D1.-; no longer D1.C
Changed lines of the file:
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@@
 <?xml version="1.0" encoding="utf-8"?>
 <!DOCTYPE eagle SYSTEM "eagle.dtd">
-<eagle version="8.2.2">
+<eagle version="8.3.2">
 <drawing>
 <settings>
 <setting alwaysvectorfont="no"/>
+<setting keepoldvectorfont="yes"/>
 <setting verticaltext="up"/>
 </settings>
@@
 <attribute name="VALUE" x="60.0964" y="38.5064" size="1.27" layer="28" rot="MR270"/>
 </element>
-<element name="R12" library="CalvEngIO-Passives" package="R0402" value="1.5M" x="66.5226" y="43.6118" smashed="yes" rot="MR270">
+<element name="R12" library="CalvEngIO-Passives" package="R0402" value="1.47M" x="66.5226" y="43.6118" smashed="yes" rot="MR270">
 <attribute name="NAME" x="65.7606" y="45.7454" size="0.6096" layer="26" rot="MR180"/>
 <attribute name="VALUE" x="68.4276" y="44.2468" size="1.27" layer="28" rot="MR270"/>
 </element>
-<element name="R1" library="CalvEngIO-Passives" package="R0402" value="205" x="54.5338" y="40.259" smashed="yes" rot="MR0.1">
+<element name="R1" library="CalvEngIO-Passives" package="R0402" value="105" x="54.5338" y="40.259" smashed="yes" rot="MR0.1">
 <attribute name="NAME" x="55.06480625" y="38.886203125" size="0.6096" layer="26" rot="MR0.1"/>
 <attribute name="VALUE" x="55.165475" y="38.35289375" size="1.27" layer="28" rot="MR0.1"/>
@@
 <attribute name="VALUE" x="49.9423625" y="34.42336875" size="0.4064" layer="28" rot="MR90.2"/>
 </element>
-<element name="R2" library="CalvEngIO-Passives" package="R0402" value="470" x="53.5686" y="33.3756" smashed="yes" rot="MR90">
+<element name="R2" library="CalvEngIO-Passives" package="R0402" value="487" x="53.5686" y="33.3756" smashed="yes" rot="MR90">
 <attribute name="NAME" x="54.483" y="33.274" size="0.6096" layer="26" rot="MR90"/>
 <attribute name="VALUE" x="51.6636" y="32.7406" size="1.27" layer="28" rot="MR90"/>
@@
 <attribute name="VALUE" x="58.3438" y="32.131" size="1.27" layer="28" rot="MR90"/>
 </element>
-<element name="R8" library="CalvEngIO-Passives" package="R0402" value="210k" x="55.4228" y="29.718" smashed="yes" rot="MR0">
+<element name="R8" library="CalvEngIO-Passives" package="R0402" value="205k" x="55.4228" y="29.718" smashed="yes" rot="MR0">
 <attribute name="NAME" x="53.975" y="29.5402" size="0.6096" layer="26" rot="MR0"/>
 <attribute name="VALUE" x="56.0578" y="27.813" size="1.27" layer="28" rot="MR0"/>
 </element>
-<element name="R9" library="CalvEngIO-Passives" package="R0402" value="210k" x="55.3974" y="31.2928" smashed="yes" rot="MR180">
+<element name="R9" library="CalvEngIO-Passives" package="R0402" value="205k" x="55.3974" y="31.2928" smashed="yes" rot="MR180">
 <attribute name="NAME" x="52.9082" y="31.5468" size="0.6096" layer="26" rot="MR180"/>
 <attribute name="VALUE" x="54.7624" y="33.1978" size="1.27" layer="28" rot="MR180"/>
@@
 <attribute name="VALUE" x="75.946" y="19.9136" size="0.6096" layer="28" ratio="20" rot="MR270" align="top-center"/>
 </element>
-<element name="D1" library="CalvEngIO-DiscreteSemi" package="SOD-323" value="" x="62.23" y="43.0784" smashed="yes" rot="MR270">
-<attribute name="NAME" x="61.7474" y="41.1226" size="0.6096" layer="26" rot="MR180"/>
-<attribute name="PROD_ID" value="DIO-09646" x="62.23" y="43.0784" size="1.778" layer="28" rot="MR270" display="off"/>
-<attribute name="VALUE" value="" x="66.04" y="45.6184" size="1.27" layer="28" rot="MR270"/>
+<element name="D1" library="CalvEngIO-DiscreteSemi" package="USC" value="" x="62.23" y="43.0784" smashed="yes" rot="MR90">
+<attribute name="NAME" x="62.7126" y="45.0342" size="0.6096" layer="26" rot="MR0"/>
 </element>
 <element name="AMP" library="CalvEngIO-AnalogIC" package="TSSOP14" value="OP-QUAD-TSSOP14" x="62.992" y="36.9824" smashed="yes" rot="MR90">
@@
 </element>
 <element name="U$1" library="CalvEngIO-Logos" package="CALVENGIO_HANDLE.05" value="CALVENGIO_HANDLEHANDLE.05" x="50.4952" y="15.24"/>
+<element name="U$2" library="CalvEngIO-Logos" package="REV.F" value="REVISION.F" x="35.1282" y="1.3716" rot="MR0"/>
 </elements>
 <signals>
@@
 </signal>
 <signal name="N$10">
-<contactref element="D1" pad="A"/>
+<contactref element="D1" pad="+"/>
 <contactref element="AMP" pad="9"/>
 <contactref element="AMP" pad="8"/>
@@
 <contactref element="R12" pad="1"/>
 <contactref element="C10" pad="2"/>
-<contactref element="D1" pad="C"/>
+<contactref element="D1" pad="-"/>
 <contactref element="AMP" pad="13"/>
 <contactref element="BREAKOUT" pad="3"/>
@@
 <wire x1="51.943" y1="51.4096" x2="50.7746" y2="52.578" width="0.3048" layer="1"/>
 <wire x1="50.7746" y1="52.578" x2="50.7746" y2="56.769" width="0.3048" layer="1"/>
-<wire x1="62.1954" y1="44.384" x2="64.3636" y2="44.384" width="0.3048" layer="16"/>
-<wire x1="62.1954" y1="44.384" x2="62.23" y2="44.2284" width="0.3048" layer="16"/>
+<wire x1="62.2208" y1="44.3586" x2="64.3636" y2="44.384" width="0.3048" layer="16"/>
+<wire x1="62.2208" y1="44.3586" x2="62.23" y2="44.2284" width="0.3048" layer="16"/>
 <wire x1="64.3636" y1="44.384" x2="66.4004" y2="44.384" width="0.3048" layer="16"/>
 <wire x1="66.4004" y1="44.384" x2="66.5226" y2="44.2618" width="0.3048" layer="16"/>
